File: hardware/scHnRk/scHnRk_3.brd (EAGLE design)
At the start: 100 x 47.6 mm, 47 parts, among them IC1 ATTINY87/167AUTOMOTIVETSSOP, SW1 L_BUTTON, SW2 R_BUTTON, SW3 RESET, SW4 SSAJ120100, U2 MCP1825S-5002E/DB, U3 PMV32UP

Commit message: added new revisions
Parts:
- removed C5, C6: 9pF, adafruit:C0603K
- removed JP4: (no value), SparkFun-Connectors:1X09
- removed U$3: 16MHZ-2467444, scHnRk:16MHZ-2467444
- removed U3: PMV32UP, NXP_By_element14_Batch_1:SOT95P230X110-3N
- added C3, C4: 9pF, adafruit:C0603K
- added JP3: (no value), SparkFun-Connectors:1X09
- added U1: MCP1825S-5002E/DB, Microchip_By_element14_Batch_1:SOT230P700X180-4N
- added XTAL1: 16MHZ-2467444, scHnRk:16MHZ-2467444
- C1, C2: device adafruit:C1206K -> SparkFun-Passives:0805
- D1: value 3.6 Zener -> B0520LW-7-F; device adafruit:SOD-523 -> adafruit:SOD-123
- D3: value B0520LW-7-F -> 3.6 Zener; device adafruit:SOD-123 -> adafruit:SOD-523
- R1: value 66.5 -> 180R
- R2: value 66.5 -> 1K5
- R3: value 1K5 -> 180R
- R4, R5: value 180R -> 66.5
- SW1: value L_BUTTON -> SSAJ120100; device scHnRk:SKRBAGE010 -> scHnRk:SSAJ120100
- SW2: value R_BUTTON -> L_BUTTON
- SW3: value RESET -> R_BUTTON
- SW4: value SSAJ120100 -> RESET; device scHnRk:SSAJ120100 -> scHnRk:SKRBAGE010
- U2: value MCP1825S-5002E/DB -> PMV32UP; device Microchip_By_element14_Batch_1:SOT230P700X180-4N -> NXP_By_element14_Batch_1:SOT95P230X110-3N
- moved H3 90.2 mm to (4.92, 5.71)
- moved H8 90.2 mm to (86.7, 5.71)
- moved H1 39.9 mm to (39.8, 5.71)
- moved H6 39.9 mm to (51.8, 43.8)
- moved H4 38.1 mm to (86.7, 43.8)
- moved H7 38.1 mm to (4.92, 43.8)
- moved SW2 34.3 mm to (78.4, 41.9)
- moved SW4 30.4 mm to (62.9, 24.1), turned to 270 degrees
- moved SJ4 26.7 mm to (76.8, 11.4)
- moved SJ2 24.4 mm to (76.8, 38.1), turned to 0 degrees
- moved SW3 22.7 mm to (78.4, 7.62), turned to 90 degrees
- moved R3 16.2 mm to (86.4, 12.7), turned to 90 degrees
- moved R1 15.1 mm to (89.5, 12.7), turned to 90 degrees
- moved R4 15.1 mm to (82.5, 26.0), turned to 180 degrees
- moved SW1 13.1 mm to (90.5, 36.8)
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- renumbered U$1 to BATT1, U$2 to BATT2
Connections:
- net 5V: now also JP3.1, R2.2, U2.3; no longer JP4.1, R3.2, U3.3
- net D0/SCA/LED: now also JP3.8, SJ3.2; no longer JP4.8, SJ2.2
- net D1/LB: now also JP3.7, SJ4.1; no longer JP4.7, SJ3.1
- net D2/SCL: now also JP3.6; no longer JP4.6
- net D3: now also JP3.5, R4.2; no longer JP4.5, R1.2
- net D4/A4: now also JP3.4, R5.2; no longer JP4.4, R2.2
- net D6/A6/RB: now also SJ2.1; no longer SJ4.1
- net GND: now also C3.2, C4.2, D3.A, H4.B3,6, JP3.2, JP3.9, R1.1, R3.1, SW4.P$4, U1.2, U1.4; no longer C5.2, C6.2, D1.A, H3.B3,6, JP4.2, JP4.9, R4.1, R5.1, SW1.P$4, U2.2, U2.4
- net N$10: now also D3.K; no longer D2.K
- net N$15: now also R2.1, R4.1; no longer R1.1, R3.1
- net N$16: now also R5.1; no longer R2.1
- net N$2: now also SJ2.2, SW2.P$1, SW2.P$3; no longer SJ4.2, SW1.P$1, SW1.P$3
- net N$22: now also U2.2; no longer U3.2
- net N$28: now also R1.2; no longer R4.2
- net N$29: now also R3.2; no longer R5.2
- net N$34: now also SJ3.1; no longer SJ2.1
- net N$7: now also SW1.P$C, U2.1; no longer SW4.P$C, U3.1
- net N$8: now also SJ4.2, SW3.P$1, SW3.P$3; no longer SJ3.2, SW2.P$1, SW2.P$3
- net N$9: now also D2.K; no longer D1.K
- net PRE5V: now also D1.C, SW1.P$1, U1.3; no longer D3.C, SW4.P$1, U2.3
- net RESET: now also JP3.3, SW4.P$1, SW4.P$3; no longer JP4.3, SW3.P$1, SW3.P$3
- net USBVCC: now also D1.A; no longer D3.A
- net VBATT: now also U1.1; no longer U2.1
- net XTAL1: now also C3.1, XTAL1.P$1; no longer C5.1, U$3.P$1
- net XTAL2: now also C4.1, XTAL1.P$3; no longer C6.1, U$3.P$3
Routing:
- net GND: track 286.6 -> 282.5 mm
- net D12/A12/SS: track 21.0 -> 25.1 mm
- net 5V: track 138.4 -> 140.8 mm
- net D13/A13: track 35.0 -> 37.2 mm
- net D4/A4: track 37.5 -> 36.9 mm
- net D3: track 33.6 -> 34.2 mm
- net D0/SCA/LED: track 24.5 -> 25.1 mm
- net RESET: track 26.2 -> 25.6 mm
Other:
- board text added: "ScHnRk v0.3"
- board text removed: "ScHnRk v0.2"
