File: hardware/scHnRk/scHnRk_4.sch (EAGLE design)
At the start: 47 parts, among them IC1 ATTINY87/167AUTOMOTIVETSSOP, SW1 SSAJ120100, SW2 L_BUTTON, SW3 R_BUTTON, SW4 RESET, U1 MCP1825S-5002E/DB, U2 PMV32UP

Commit message: added new revisions
Parts:
- C1, C2: value 10uF -> 9pF; device SparkFun-Passives:CAP0805 -> SparkFun-Passives:CAP0603-CAP
- C3, C4: value 9pF -> 10uF; device adafruit:C-USC0603K -> SparkFun-Passives:CAP0805
- JP1: value USBPCB -> (none); device SparkFun-Connectors:USBPCB -> SparkFun-Connectors:M09
- JP3: value (none) -> USBPCB; device SparkFun-Connectors:M09 -> SparkFun-Connectors:USBPCB
- LED3: value WS2812B5050 -> PWR; device adafruit:WS2812B5050 -> adafruit:LEDCHIPLED_0603
- LED4: value WS2812B5050 -> D1; device adafruit:WS2812B5050 -> adafruit:LEDCHIPLED_0603
- LED6: value PWR -> WS2812B5050; device adafruit:LEDCHIPLED_0603 -> adafruit:WS2812B5050
- LED7: value D1 -> WS2812B5050; device adafruit:LEDCHIPLED_0603 -> adafruit:WS2812B5050
- R1: value 180R -> 1K5; device adafruit:R-US_R0603 -> SparkFun-Passives:RESISTOR0805-RES
- R2: value 1K5 -> 66.5; device adafruit:R-US_R0603 -> SparkFun-Passives:RESISTOR0603-RES
- R3: value 180R -> 66.5; device adafruit:R-US_R0603 -> SparkFun-Passives:RESISTOR0603-RES
- R4, R5: value 66.5 -> 180R; device adafruit:R-US_R0603 -> SparkFun-Passives:RESISTOR0805-RES
- renumbered SJ1 to J5, SJ2 to J1, SJ3 to J6, SJ4 to J2, SJ5 to J3, SJ6 to J4
Connections:
- net 5V: now also C4.1, JP2.1, LED6.VDD, LED7.VDD, R1.2; no longer C2.1, JP3.1, LED3.VDD, LED4.VDD, R2.2
- net D0/SCA/LED: now also JP2.8; no longer JP3.8
- net D1/LB: now also JP2.7; no longer JP3.7
- net D10/A10/MOSI: now also JP1.4; no longer JP2.4
- net D11/A11/SCK: now also JP1.3; no longer JP2.3
- net D12/A12/SS: now also JP1.2; no longer JP2.2
- net D13/A13: now also JP1.1; no longer JP2.1
- net D2/SCL: now also JP2.6; no longer JP3.6
- net D3: now also JP2.5, R2.2; no longer JP3.5, R4.2
- net D4/A4: now also JP2.4, R3.2; no longer JP3.4, R5.2
- net D6/A6/RB: now also JP1.8; no longer JP2.8
- net D7/A7: now also JP1.7; no longer JP2.7
- net D8/A8/MISO: now also JP1.6; no longer JP2.6
- net D9/A9: now also JP1.5; no longer JP2.5
- net GND: now also H5.MOUNT, H6.MOUNT, H8.MOUNT, JP2.2, JP2.9, JP3.GND, LED6.GND, LED7.GND, R4.1, R5.1; no longer H2.MOUNT, H4.MOUNT, JP1.GND, JP3.2, JP3.9, LED3.GND, LED4.GND, R1.1, R3.1
- net N$15: now also JP3.D-, R1.1; no longer JP1.D-, R4.1
- net N$16: now also JP3.D+, R3.1; no longer JP1.D+, R5.1
- net N$28: now also LED3.C, R4.2; no longer LED6.C, R1.2
- net N$29: now also LED4.C, R5.2; no longer LED7.C, R3.2
- net N$31: now also LED3.A; no longer LED6.A
- net N$34: now also LED4.A; no longer LED7.A
- net N$4: now also LED5.DI; no longer LED3.DI
- net N$5: now also LED5.DO, LED6.DI; no longer LED3.DO, LED4.DI
- net N$6: now also LED6.DO, LED7.DI; no longer LED4.DO, LED5.DI
- net RESET: now also JP2.3; no longer JP3.3
- net USBVCC: now also JP3.VBUS; no longer JP1.VBUS
- net VBATT: now also C3.1, JP1.9; no longer C1.1, JP2.9
- net XTAL1: now also C1.1; no longer C3.1
- net XTAL2: now also C2.1; no longer C4.1
Other:
- moved on the sheet: C1, C2, C3, C4, H2, H3, H4, H5, H6, H7, JP2, R1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
