File: hardware/scHnRk_6.sch (EAGLE design)
At the start: 48 parts, among them IC1 ATTINY87/167AUTOMOTIVETSSOP, J1 JUMPER, J2 JUMPER, J3 JUMPER, J4 JUMPER, J5 JUMPER, J6 JUMPER, SW1 SSAJ120100, SW2 L_BUTTON, SW3 R_BUTTON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

Commit message: added skeletons, transiting to atmega328p-mu
Parts:
- removed IC1: ATTINY87/167AUTOMOTIVETSSOP, attiny87_167_automotive:ATTINY87/167AUTOMOTIVETSSOP
- removed JP1, JP2: (no value), SparkFun-Connectors:M09
- removed XTAL1: 16MHZ-2467444, scHnRk:16MHZ-2467444
- added JP4: FTDI_DEVICE, SparkFun-Connectors:FTDI_DEVICE
- added JP5: (no value), SparkFun-Connectors:I2C_STANDARD
- added JP6, JP7: (no value), SparkFun-Connectors:M12PTH
- added R7: 10k, SparkFun-Passives:RESISTOR0805-RES
- added U$1: 16MHZ, SparkFun-FreqCtrl:RESONATOR16MHZ
- added U4: ATMEGA328P-MU, Atmel_By_element14_Batch_1-00:ATMEGA328P-MU
- C1, C2: value 9pF -> 0.1uF; device SparkFun-Passives:CAP0603-CAP -> SparkFun-Passives:CAP0805
Connections:
- removed net D0/SCA/LED: IC1.(PCINT8/OC1AU/DI/SDA)PB0, J6.2, JP2.8
- removed net D1/LB: IC1.(PCINT9/OC1BU/DO)PB1, J2.1, JP2.7
- removed net D10/A10/MOSI: IC1.(MOSI/SDA/DI/ADC4/PCINT4)PA4, JP1.4
- removed net D11/A11/SCK: IC1.(SCK/SCL/USCK/T1/ADC5/PCINT5)PA5, JP1.3
- removed net D12/A12/SS: IC1.(!SS!/AIN0/ADC6/PCINT6)PA6, JP1.2
- removed net D13/A13: IC1.(AREF/XREF/AIN1/ADC7/PCINT7)PA7, JP1.1, LED1.DI
- removed net D2/SCL: IC1.(PCINT10/OC1AV/USCK/SCL)PB2, JP2.6
- removed net D4/A4: IC1.(PCINT14/ADC9/OC1AX/INT0)PB6, JP2.4, R3.2
- removed net D6/A6/RB: IC1.(RXLIN/RXD/ADC0/PCINT0)PA0, J1.1, JP1.8
- removed net D7/A7: IC1.(TXLIN/TXD/ADC1/PCINT1)PA1, JP1.7
- removed net D8/A8/MISO: IC1.(MISO/DO/OC0A/ADC2/PCINT2)PA2, JP1.6
- removed net D9/A9: IC1.(INT1/ISRC/ADC3/PCINT3)PA3, JP1.5
- new net A0: U4.PC0
- new net A1: U4.PC1
- new net A2: U4.PC2
- new net A3: U4.PC3
- new net A4/SDA: JP5.3, U4.PC4
- new net A5/SCL: JP5.4, U4.PC5
- new net A6: U4.ADC6
- new net A7: U4.ADC7
- new net D0/RXD: JP4.TXO, JP7.1, U4.PD0
- new net D1/TXD: JP4.RXI, JP7.2, U4.PD1
- new net D10: U4.PB2
- new net D11/MOSI: U4.PB3
- new net D12/MISO: U4.PB4
- new net D13/SCK: J6.2, U4.PB5
- new net D2: R3.2, U4.PD2
- new net D4: JP7.4, U4.PD4
- new net D5: JP7.5, U4.PD5
- new net D6: JP7.6, U4.PD6
- new net D7: R2.2, U4.PD7
- new net D8: JP7.7, U4.PB0
- new net D9: U4.PB1
- new net HEATSINK: U4.EP
- new net N$21: JP7.12
- new net N$23: JP7.11
- new net N$25: C2.2, JP4.DTR
- new net N$256: JP6.12
- new net N$26: LED1.DI
- new net N$264: JP6.11
- new net N$265: JP6.10
- new net N$266: JP6.9
- new net N$267: JP6.8
- new net N$268: JP6.7
- new net N$269: JP6.6
- new net N$271: JP6.5
- new net N$272: JP6.4
- new net N$273: JP6.3
- new net N$274: JP6.2
- new net N$285: JP6.1
- new net N$307: J1.1
- new net N$308: J2.1
- new net N$62: C1.2, U4.AREF
- new net N$81: JP7.10
- new net N$84: JP7.9
- new net N$85: JP7.8
- net 5V: now also JP4.VCC, JP5.2, R7.1, U4.AVCC, U4.VCC, U4.VCC_2; no longer IC1.AVCC, IC1.VCC, JP2.1
- net D3: now also JP7.3, U4.PD3; no longer IC1.(PCINT11/OC1BV)PB3, JP2.5, R2.2
- net GND: now also C1.1, JP4.CTS, JP4.GND, JP5.1, U$1.2, U4.GND, U4.GND_2, U4.GND_3; no longer C1.2, C2.2, H5.MOUNT, H6.MOUNT, H8.MOUNT, IC1.AGND, IC1.GND, JP2.2, JP2.9
- net RESET: now also C2.1, R7.2, U4.PC6; no longer IC1.(PCINT15/ADC10/OC1BX/!RESET!/DW)PB7, JP2.3
- net VBATT: no longer JP1.9
- net XTAL1: now also U$1.3, U4.PB6; no longer C1.1, IC1.(PCINT12/OC1AW/XTAL1/CLKI)PB4, XTAL1.P$1
- net XTAL2: now also U$1.1, U4.PB7; no longer C2.1, IC1.(PCINT13/ADC8/OC1BW/XTAL2/CLKO)PB5, XTAL1.P$2
Other:
- moved on the sheet: C1, C2, D1, D2, D3, F1, J1, J2, J3, J4, J5, J6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
